File: KiCad/Power.kicad_sch (KiCad schematic)
At the start: 0 parts

Commit message: he afegit la part de potencia
Parts:
- added C1, C2, C5, C6: 10u, symbol Device:C_Polarized
- added C3, C4: 0.1u, symbol Device:C
- added D1: STZ5_6N, symbol Device:D_Zener
- added J1, J2: Conn_01x02_Pin, symbol Connector:Conn_01x02_Pin
- added Q1: 2SD600, Package_TO_SOT_THT:TO-126-3_Vertical, symbol Transistor_BJT:2SD600
- added R1: 210, symbol Device:R
- added R2: 130, symbol Device:R
- added R3: 330, symbol Device:R
- added R4: 1K, symbol Device:R
- added U1: LM1117S-ADJ, Package_TO_SOT_SMD:TO-263-3_TabPin2, symbol Regulator_Linear:LM1117S-ADJ
- added U6: LM1117DT-3.3, Package_TO_SOT_SMD:TO-252-3_TabPin2, symbol Regulator_Linear:LM1117DT-3.3
- added U7: TSR1-2450E, Converter_DCDC:Converter_DCDC_TRACO_TSR1-xxxxE_THT, symbol Converter_DCDC:TSR1-2450E
Connections:
- new net: C3.1, C5.1, J1.1 (Pin_1), Q1.2 (C), R3.1
- new net: R1.1, R2.2, U1.1 (ADJ)
- new net: D1.1 (K), Q1.3 (B), R3.2
- new net +12V: U7.1 (Vin)
- new net GND: C1.2, C2.2, C3.2, C4.2, C5.2, C6.2, D1.2 (A), J1.2 (Pin_2), J2.2 (Pin_2), R1.2, R4.2, U6.1 (GND)
- new net VCC: C2.1, R2.1, U1.2 (VO), U6.2 (VO)
- new net Vout_DC/DC: C1.1, C4.1, C6.1, J2.1 (Pin_1), Q1.1 (E), R4.1, U1.3 (VI), U6.3 (VI), U7.3 (Vout)
Other:
- note added: "ETAPA DE PÓTENCIA"
- note added: "REGULADOR DC/DC 5V"
- note added: "REGULADOR DE TENSIÓ 3.3V"

Commit message: afegit part analogica
Parts:
- renumbered C1 to C?, C2 to C?, C5 to C?, C3 to C?, C6 to C?, C4 to C?, D1 to D?, J2 to J?, J1 to J?, Q1 to Q?, R4 to R?, R1 to R?, R2 to R?, R3 to R?, U6 to U?, U1 to U?, U7 to U?
Connections:
- net Vbat: now reaches C?.1, C?.1, J?.1 (Pin_1), Q?.2 (C), R?.1
Changed lines of the file:
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@@
+		)
+	)
+	(global_label "Vbat"
+		(shape input)
+		(at 31.75 88.9 180)
+		(fields_autoplaced yes)
+		(effects
+			(font
+				(size 1.27 1.27)
+			)
+			(justify right)
+		)
+		(property "Intersheetrefs" "${INTERSHEET_REFS}"
+			(at 24.6525 88.9 0)
+			(effects
+				(font
+					(size 1.27 1.27)
+				)
+				(justify right)
+				(hide yes)
+			)
 		)
 	)
@@
 		(dnp no)
 		(fields_autoplaced yes)
-		(property "Reference" "R4"
+		(property "Reference" "R?"
 			(at 111.76 96.5199 0)
 			(effects
@@
 		)
 		(instances
+			(project "projecte_sostre"
+				(path "/12dc51a9-2603-4518-b497-f55f3848c2a7/34d9cf6f-a994-4628-b3ba-09455bb98cce"
+					(reference "R?")
+					(unit 1)
+				)
+			)
 			(project "Power"
 				(path "/f7c86f09-5bbf-4c4b-85ef-97cdf0efc1c7"
@@
 		(dnp no)
 		(fields_autoplaced yes)
-		(property "Reference" "C1"
+		(property "Reference" "C?"
 			(at 44.45 46.1009 0)
 			(effects
@@
 		)
 		(instances
+			(project "projecte_sostre"
+				(path "/12dc51a9-2603-4518-b497-f55f3848c2a7/34d9cf6f-a994-4628-b3ba-09455bb98cce"
+					(reference "C?")
+					(unit 1)
+				)
+			)
 			(project "Power"
 				(path "/f7c86f09-5bbf-4c4b-85ef-97cdf0efc1c7"
@@
 		(dnp no)
 		(fields_autoplaced yes)
-		(property "Reference" "U6"
+		(property "Reference" "U?"
 			(at 93.98 161.29 0)
 			(effects
@@
 		)
 		(instances
+			(project "projecte_sostre"
+				(path "/12dc51a9-2603-4518-b497-f55f3848c2a7/34d9cf6f-a994-4628-b3ba-09455bb98cce"
+					(reference "U?")
+					(unit 1)
+				)
+			)
 			(project "Power"
 				(path "/f7c86f09-5bbf-4c4b-85ef-97cdf0efc1c7"
@@
 		(dnp no)
 		(fields_autoplaced yes)
-		(property "Reference" "C2"
+		(property "Reference" "C?"
 			(at 82.55 39.7509 0)
 			(effects
@@
 		)
 		(instances
+			(project "projecte_sostre"
+				(path "/12dc51a9-2603-4518-b497-f55f3848c2a7/34d9cf6f-a994-4628-b3ba-09455bb98cce"
+					(reference "C?")
+					(unit 1)
+				)
+			)
 			(project "Power"
 				(path "/f7c86f09-5bbf-4c4b-85ef-97cdf0efc1c7"
@@
 		(dnp no)
 		(fields_autoplaced yes)
-		(property "Reference" "#PWR01"
+		(property "Reference" "#PWR?"
 			(at 29.21 175.26 0)
 			(effects
@@
 		)
 		(instances
+			(project "projecte_sostre"
+				(path "/12dc51a9-2603-4518-b497-f55f3848c2a7/34d9cf6f-a994-4628-b3ba-09455bb98cce"
+					(reference "#PWR?")
+					(unit 1)
+				)
+			)
 			(project "Power"
 				(path "/f7c86f09-5bbf-4c4b-85ef-97cdf0efc1c7"
@@
 		(dnp no)
 		(fields_autoplaced yes)
-		(property "Reference" "J2"
+		(property "Reference" "J?"
 			(at 121.285 91.44 0)
 			(effects
@@
 		)
 		(instances
+			(project "projecte_sostre"
+				(path "/12dc51a9-2603-4518-b497-f55f3848c2a7/34d9cf6f-a994-4628-b3ba-09455bb98cce"
+					(reference "J?")
+					(unit 1)
+				)
+			)
 			(project "Power"
 				(path "/f7c86f09-5bbf-4c4b-85ef-97cdf0efc1c7"
@@
 		(dnp no)
 		(fields_autoplaced yes)
-		(property "Reference" "C5"
+		(property "Reference" "C?"
 			(at 46.99 95.6309 0)
 			(effects
@@
 		)
 		(instances
+			(project "projecte_sostre"
+				(path "/12dc51a9-2603-4518-b497-f55f3848c2a7/34d9cf6f-a994-4628-b3ba-09455bb98cce"
+					(reference "C?")
+					(unit 1)
+				)
+			)
 			(project "Power"
 				(path "/f7c86f09-5bbf-4c4b-85ef-97cdf0efc1c7"
@@
 		(dnp no)
 		(fields_autoplaced yes)
-		(property "Reference" "#PWR03"
+		(property "Reference" "#PWR?"
 			(at 72.39 115.57 0)
 			(effects
@@
 		)
 		(instances
+			(project "projecte_sostre"
+				(path "/12dc51a9-2603-4518-b497-f55f3848c2a7/34d9cf6f-a994-4628-b3ba-09455bb98cce"
+					(reference "#PWR?")
+					(unit 1)
+				)
+			)
 			(project "Power"
 				(path "/f7c86f09-5bbf-4c4b-85ef-97cdf0efc1c7"
@@
 		(dnp no)
 		(fields_autoplaced yes)
-		(property "Reference" "R1"
+		(property "Reference" "R?"
 			(at 69.85 54.6099 0)
 			(effects
@@
 		)
 		(instances
+			(project "projecte_sostre"
+				(path "/12dc51a9-2603-4518-b497-f55f3848c2a7/34d9cf6f-a994-4628-b3ba-09455bb98cce"
+					(reference "R?")
+					(unit 1)
+				)
+			)
 			(project "Power"
 				(path "/f7c86f09-5bbf-4c4b-85ef-97cdf0efc1c7"
@@
 		(dnp no)
 		(fields_autoplaced yes)
-		(property "Reference" "J1"
+		(property "Reference" "J?"
 			(at 19.685 93.98 0)
 			(effects
@@
 		)
 		(instances
+			(project "projecte_sostre"
+				(path "/12dc51a9-2603-4518-b497-f55f3848c2a7/34d9cf6f-a994-4628-b3ba-09455bb98cce"
+					(reference "J?")
+					(unit 1)
+				)
+			)
 			(project "Power"
 				(path "/f7c86f09-5bbf-4c4b-85ef-97cdf0efc1c7"
@@
 		(on_board yes)
 		(dnp no)
-		(property "Reference" "C3"
+		(property "Reference" "C?"
 			(at 57.15 96.5199 0)
 			(effects
@@
 		)
 		(instances
+			(project "projecte_sostre"
+				(path "/12dc51a9-2603-4518-b497-f55f3848c2a7/34d9cf6f-a994-4628-b3ba-09455bb98cce"
+					(reference "C?")
+					(unit 1)
+				)
+			)
 			(project "Power"
 				(path "/f7c86f09-5bbf-4c4b-85ef-97cdf0efc1c7"
@@
 		(dnp no)
 		(fields_autoplaced yes)
-		(property "Reference" "R2"
+		(property "Reference" "R?"
 			(at 69.85 40.6399 0)
 			(effects
@@
 		)
 		(instances
+			(project "projecte_sostre"
+				(path "/12dc51a9-2603-4518-b497-f55f3848c2a7/34d9cf6f-a994-4628-b3ba-09455bb98cce"
+					(reference "R?")
+					(unit 1)
+				)
+			)
 			(project "Power"
 				(path "/f7c86f09-5bbf-4c4b-85ef-97cdf0efc1c7"
@@
 		(dnp no)
 		(fields_autoplaced yes)
-		(property "Reference" "Q1"
+		(property "Reference" "Q?"
 			(at 72.39 82.55 90)
 			(effects
@@
 		)
 		(instances
+			(project "projecte_sostre"
+				(path "/12dc51a9-2603-4518-b497-f55f3848c2a7/34d9cf6f-a994-4628-b3ba-09455bb98cce"
+					(reference "Q?")
+					(unit 1)
+				)
+			)
 			(project "Power"
 				(path "/f7c86f09-5bbf-4c4b-85ef-97cdf0efc1c7"
@@
 		(dnp no)
 		(fields_autoplaced yes)
-		(property "Reference" "#PWR02"
+		(property "Reference" "#PWR?"
 			(at 67.31 66.04 0)
 			(effects
@@
 		)
 		(instances
+			(project "projecte_sostre"
+				(path "/12dc51a9-2603-4518-b497-f55f3848c2a7/34d9cf6f-a994-4628-b3ba-09455bb98cce"
+					(reference "#PWR?")
+					(unit 1)
+				)
+			)
 			(project "Power"
 				(path "/f7c86f09-5bbf-4c4b-85ef-97cdf0efc1c7"
@@
 		(dnp no)
 		(fields_autoplaced yes)
-		(property "Reference" "C6"
+		(property "Reference" "C?"
 			(at 93.98 95.6309 0)
 			(effects
@@
 		)
 		(instances
+			(project "projecte_sostre"
+				(path "/12dc51a9-2603-4518-b497-f55f3848c2a7/34d9cf6f-a994-4628-b3ba-09455bb98cce"
+					(reference "C?")
+					(unit 1)
+				)
+			)
 			(project "Power"
 				(path "/f7c86f09-5bbf-4c4b-85ef-97cdf0efc1c7"
@@
 		(dnp no)
 		(fields_autoplaced yes)
-		(property "Reference" "C4"
+		(property "Reference" "C?"
 			(at 102.87 96.5199 0)
 			(effects
@@
 		)
 		(instances
+			(project "projecte_sostre"
+				(path "/12dc51a9-2603-4518-b497-f55f3848c2a7/34d9cf6f-a994-4628-b3ba-09455bb98cce"
+					(reference "C?")
+					(unit 1)
+				)
+			)
 			(project "Power"
 				(path "/f7c86f09-5bbf-4c4b-85ef-97cdf0efc1c7"
@@
 		(dnp no)
 		(fields_autoplaced yes)
-		(property "Reference" "#PWR04"
+		(property "Reference" "#PWR?"
 			(at 93.98 181.61 0)
 			(effects
@@
 		)
 		(instances
+			(project "projecte_sostre"
+				(path "/12dc51a9-2603-4518-b497-f55f3848c2a7/34d9cf6f-a994-4628-b3ba-09455bb98cce"
+					(reference "#PWR?")
+					(unit 1)
+				)
+			)
 			(project "Power"
 				(path "/f7c86f09-5bbf-4c4b-85ef-97cdf0efc1c7"
@@
 		(dnp no)
 		(fields_autoplaced yes)
-		(property "Reference" "U1"
+		(property "Reference" "U?"
 			(at 53.34 30.48 0)
 			(effects
@@
 		)
 		(instances
+			(project "projecte_sostre"
+				(path "/12dc51a9-2603-4518-b497-f55f3848c2a7/34d9cf6f-a994-4628-b3ba-09455bb98cce"
+					(reference "U?")
+					(unit 1)
+				)
+			)
 			(project "Power"
 				(path "/f7c86f09-5bbf-4c4b-85ef-97cdf0efc1c7"
@@
 		(dnp no)
 		(fields_autoplaced yes)
-		(property "Reference" "#PWR06"
+		(property "Reference" "#PWR?"
 			(at 40.64 58.42 0)
 			(effects
@@
 		)
 		(instances
+			(project "projecte_sostre"
+				(path "/12dc51a9-2603-4518-b497-f55f3848c2a7/34d9cf6f-a994-4628-b3ba-09455bb98cce"
+					(reference "#PWR?")
+					(unit 1)
+				)
+			)
 			(project "Power"
 				(path "/f7c86f09-5bbf-4c4b-85ef-97cdf0efc1c7"
@@
 		(dnp no)
 		(fields_autoplaced yes)
-		(property "Reference" "#PWR05"
+		(property "Reference" "#PWR?"
 			(at 78.74 52.07 0)
 			(effects
@@
 		)
 		(instances
+			(project "projecte_sostre"
+				(path "/12dc51a9-2603-4518-b497-f55f3848c2a7/34d9cf6f-a994-4628-b3ba-09455bb98cce"
+					(reference "#PWR?")
+					(unit 1)
+				)
+			)
 			(project "Power"
 				(path "/f7c86f09-5bbf-4c4b-85ef-97cdf0efc1c7"
@@
 		(dnp no)
 		(fields_autoplaced yes)
-		(property "Reference" "R3"
+		(property "Reference" "R?"
 			(at 66.04 92.7099 0)
 			(effects
@@
 		)
 		(instances
+			(project "projecte_sostre"
+				(path "/12dc51a9-2603-4518-b497-f55f3848c2a7/34d9cf6f-a994-4628-b3ba-09455bb98cce"
+					(reference "R?")
+					(unit 1)
+				)
+			)
 			(project "Power"
 				(path "/f7c86f09-5bbf-4c4b-85ef-97cdf0efc1c7"
@@
 		(on_board yes)
 		(dnp no)
-		(property "Reference" "D1"
+		(property "Reference" "D?"
 			(at 74.93 100.3299 90)
 			(effects
@@
 		)
 		(instances
+			(project "projecte_sostre"
+				(path "/12dc51a9-2603-4518-b497-f55f3848c2a7/34d9cf6f-a994-4628-b3ba-09455bb98cce"
+					(reference "D?")
+					(unit 1)
+				)
+			)
 			(project "Power"
 				(path "/f7c86f09-5bbf-4c4b-85ef-97cdf0efc1c7"
@@
 		(dnp no)
 		(fields_autoplaced yes)
-		(property "Reference" "U7"
+		(property "Reference" "U?"
 			(at 46.99 166.37 0)
 			(effects
@@
 		)
 		(instances
-			(project "Power"
-				(path "/f7c86f09-5bbf-4c4b-85ef-97cdf0efc1c7"
+			(project "projecte_sostre"
+				(path "/12dc51a9-2603-4518-b497-f55f3848c2a7/34d9cf6f-a994-4628-b3ba-09455bb98cce"
+					(reference "U?")
+					(unit 1)
+				)
+			)
+			(project "Power"
+				(path "/f7c86f09-5bbf-4c4b-85ef-97cdf0efc1c7"

Commit message: Subida para juntarlo todo 100 por 100
Other:
- moved on the sheet: U?
Changed lines of the file:
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@@
 		(effects
 			(font
-				(size 1.778 1.778)
+				(size 2.032 2.032)
 			)
 		)
@@
 	(text "ETAPA DE PÓTENCIA\n"
 		(exclude_from_sim no)
-		(at 23.622 158.75 0)
+		(at 137.922 17.78 0)
 		(effects
 			(font
-				(size 1.27 1.27)
+				(size 2.032 2.032)
 			)
 		)
@@
 		(effects
 			(font
-				(size 1.778 1.778)
+				(size 2.032 2.032)
 			)
 		)
@@
 	(wire
 		(pts
-			(xy 29.21 171.45) (xy 29.21 173.99)
+			(xy 143.51 30.48) (xy 143.51 33.02)
 		)
 		(stroke
@@
 	(wire
 		(pts
-			(xy 29.21 173.99) (xy 36.83 173.99)
+			(xy 143.51 33.02) (xy 151.13 33.02)
 		)
 		(stroke
@@
 		)
 	)
+	(polyline
+		(pts
+			(xy 184.15 62.23) (xy 231.14 62.23)
+		)
+		(stroke
+			(width 0)
+			(type default)
+		)
+	)
 	(wire
 		(pts
@@
 		)
 	)
+	(polyline
+		(pts
+			(xy 105.41 13.97) (xy 106.68 13.97)
+		)
+		(stroke
+			(width 0)
+			(type default)
+		)
+	)
 	(wire
 		(pts
@@
 		)
 	)
+	(polyline
+		(pts
+			(xy 186.69 62.23) (xy 105.41 62.23)
+		)
+		(stroke
+			(width 0)
+			(type default)
+		)
+	)
 	(wire
 		(pts
@@
 	(polyline
 		(pts
-			(xy 116.84 156.21) (xy 116.84 196.85)
+			(xy 231.14 15.24) (xy 231.14 62.23)
 		)
 		(stroke
@@
 		)
 	)
+	(wire
+		(pts
+			(xy 72.39 105.41) (xy 72.39 109.22)
+		)
+		(stroke
+			(width 0)
+			(type default)
+		)
+	)
+	(wire
+		(pts
+			(xy 109.22 101.6) (xy 109.22 109.22)
+		)
+		(stroke
+			(width 0)
+			(type default)
+		)
+	)
+	(wire
+		(pts
+			(xy 63.5 88.9) (xy 63.5 90.17)
+		)
+		(stroke
+			(width 0)
+			(type default)
+		)
+	)
+	(wire
+		(pts
+			(xy 53.34 44.45) (xy 53.34 46.99)
+		)
+		(stroke
+			(width 0)
+			(type default)
+		)
+	)
+	(wire
+		(pts
+			(xy 77.47 88.9) (xy 90.17 88.9)
+		)
+		(stroke
+			(width 0)
+			(type default)
+		)
+	)
 	(polyline
 		(pts
-			(xy 13.97 156.21) (xy 116.84 156.21)
-		)
-		(stroke
-			(width 0)
-			(type default)
-		)
-	)
-	(wire
-		(pts
-			(xy 72.39 105.41) (xy 72.39 109.22)
-		)
-		(stroke
-			(width 0)
-			(type default)
-		)
-	)
-	(wire
-		(pts
-			(xy 109.22 101.6) (xy 109.22 109.22)
-		)
-		(stroke
-			(width 0)
-			(type default)
-		)
-	)
-	(wire
-		(pts
-			(xy 63.5 88.9) (xy 63.5 90.17)
-		)
-		(stroke
-			(width 0)
-			(type default)
-		)
-	)
-	(wire
-		(pts
-			(xy 53.34 44.45) (xy 53.34 46.99)
-		)
-		(stroke
-			(width 0)
-			(type default)
-		)
-	)
-	(wire
-		(pts
-			(xy 77.47 88.9) (xy 90.17 88.9)
+			(xy 105.41 62.23) (xy 105.41 13.97)
 		)
 		(stroke
@@
 	(global_label "VCC"
 		(shape output)
-		(at 101.6 167.64 0)
+		(at 215.9 26.67 0)
 		(fields_autoplaced yes)
 		(effects
@@
 		)
 		(property "Intersheetrefs" "${INTERSHEET_REFS}"
-			(at 108.2138 167.64 0)
+			(at 222.5138 26.67 0)
 			(effects
 				(font
@@
 	(global_label "Vout_DC{slash}DC"
 		(shape output)
-		(at 57.15 173.99 0)
+		(at 171.45 33.02 0)
 		(fields_autoplaced yes)
 		(effects
@@
 		)
 		(property "Intersheetrefs" "${INTERSHEET_REFS}"
-			(at 71.6256 173.99 0)
+			(at 185.9256 33.02 0)
 			(effects
 				(font
@@
 	(global_label "Vout_DC{slash}DC"
 		(shape output)
-		(at 86.36 167.64 180)
+		(at 200.66 26.67 180)
 		(fields_autoplaced yes)
 		(effects
@@
 		)
 		(property "Intersheetrefs" "${INTERSHEET_REFS}"
-			(at 71.8844 167.64 0)
+			(at 186.1844 26.67 0)
 			(effects
 				(font
@@
 	(symbol
 		(lib_id "Regulator_Linear:LM1117DT-3.3")
-		(at 93.98 167.64 0)
+		(at 208.28 26.67 0)
 		(unit 1)
 		(exclude_from_sim no)
@@
 		(fields_autoplaced yes)
 		(property "Reference" "U?"
-			(at 93.98 161.29 0)
+			(at 208.28 20.32 0)
 			(effects
 				(font
@@
 		)
 		(property "Value" "LM1117DT-3.3"
-			(at 93.98 163.83 0)
+			(at 208.28 22.86 0)
 			(effects
 				(font
@@
 		)
 		(property "Footprint" "Package_TO_SOT_SMD:TO-252-3_TabPin2"
-			(at 93.98 167.64 0)
+			(at 208.28 26.67 0)
 			(effects
 				(font
@@
 		)
 		(property "Datasheet" "http://www.ti.com/lit/ds/symlink/lm1117.pdf"
-			(at 93.98 167.64 0)
+			(at 208.28 26.67 0)
 			(effects
 				(font
@@
 		)
 		(property "Description" "800mA Low-Dropout Linear Regulator, 3.3V fixed output, TO-252"
-			(at 93.98 167.64 0)
+			(at 208.28 26.67 0)
 			(effects
 				(font
@@
 	(symbol
 		(lib_id "power:+12V")
-		(at 29.21 171.45 0)
+		(at 143.51 30.48 0)
 		(unit 1)
 		(exclude_from_sim no)
@@
 		(fields_autoplaced yes)
 		(property "Reference" "#PWR?"
-			(at 29.21 175.26 0)
+			(at 143.51 34.29 0)
 			(effects
 				(font
@@
 		)
 		(property "Value" "+12V"
-			(at 29.21 166.37 0)
+			(at 143.51 25.4 0)
 			(effects
 				(font
@@
 		)
 		(property "Footprint" ""
-			(at 29.21 171.45 0)
+			(at 143.51 30.48 0)
 			(effects
 				(font
@@
 		)
 		(property "Datasheet" ""
-			(at 29.21 171.45 0)
+			(at 143.51 30.48 0)
 			(effects
 				(font
@@
 		)
 		(property "Description" "Power symbol creates a global label with name \"+12V\""
-			(at 29.21 171.45 0)
+			(at 143.51 30.48 0)
 			(effects
 				(font
@@
 	(symbol
 		(lib_id "power:GND")
-		(at 93.98 175.26 0)
+		(at 208.28 34.29 0)
 		(unit 1)
 		(exclude_from_sim no)
@@
 		(fields_autoplaced yes)
 		(property "Reference" "#PWR?"
-			(at 93.98 181.61 0)
+			(at 208.28 40.64 0)
 			(effects
 				(font
@@
 		)
 		(property "Value" "GND"
-			(at 93.98 180.34 0)
+			(at 208.28 39.37 0)
 			(effects
 				(font
@@
 		)
 		(property "Footprint" ""
-			(at 93.98 175.26 0)
+			(at 208.28 34.29 0)
 			(effects
 				(font
@@
 		)
 		(property "Datasheet" ""
-			(at 93.98 175.26 0)
+			(at 208.28 34.29 0)
 			(effects
 				(font
@@
 		)
 		(property "Description" "Power symbol creates a global label with name \"GND\" , ground"
-			(at 93.98 175.26 0)
+			(at 208.28 34.29 0)
 			(effects
 				(font
@@
 	(symbol
 		(lib_id "Converter_DCDC:TSR1-2450E")
-		(at 46.99 176.53 0)
+		(at 161.29 35.56 0)
 		(unit 1)
 		(exclude_from_sim no)
@@
 		(fields_autoplaced yes)
 		(property "Reference" "U?"
-			(at 46.99 166.37 0)
+			(at 161.29 25.4 0)
 			(effects
 				(font
@@
 		)
 		(property "Value" "TSR1-2450E"
-			(at 46.99 168.91 0)
+			(at 161.29 27.94 0)
 			(effects
 				(font
@@
 		)
 		(property "Footprint" "Converter_DCDC:Converter_DCDC_TRACO_TSR1-xxxxE_THT"
-			(at 46.99 182.88 0)
+			(at 161.29 41.91 0)
 			(effects
 				(font
@@
 		)
 		(property "Datasheet" "https://www.tracopower.com/products/tsr1e.pdf"
-			(at 46.99 180.34 0)
+			(at 161.29 39.37 0)
 			(effects
 				(font
@@
 		)
 		(property "Description" "1A step-down regulator, fixed 5V output voltage, 7-36V input voltage, TO-220 compatible LM78xx replacement"
-			(at 46.99 176.53 0)
-			(effects
-				(font
+			(at 161.29 35.56 0)
+			(effects
+				(font
